File: hardware/boards/glasgow/glasgow.sch (KiCad schematic (older format))
At the start: 93 parts, among them J1 USB_B_Micro, U1 CY7C68013A-56LTX, U15 TPD3S014, U2 CAT24M01W, U3 CAT24C256W, U30 ICE40HX8K-BG121, U34 ATECC508A, U36 TLV73312PQDRVRQ1, U7 LM3880MF-1AF, U8 TLV75533PDRVR, Y1 24M

Commit message: revC1-usbc: changed usb micro connector to usb type C
Parts:
- removed J1: USB_B_Micro, Connector_USB:USB_Micro-B_Molex_47346-0001, symbol Connector:USB_B_Micro
- added J1: USB_C_Receptacle_USB2.0, Connector_USB:USB_C_Receptacle_HRO_TYPE-C-31-M-12, symbol Connector:USB_C_Receptacle_USB2.0
- added R52, R53: 5k11, Resistor_SMD:R_0402_1005Metric, symbol Device:R
Connections:
- net labels added: USB_CC1, USB_CC2, VUSBIN
- wire segments 364 -> 380
- no-connect marks 8 -> 9
Other:
- moved on the sheet: C11, C12, C13, C14, C18, C19, C20, C21, C23, C24, C25, C76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

Commit message: changed level shifters, passing DRC
Parts:
- C1, C10, C11, C12, C13, C14, C15, C16, C17, C18, C19, C2, C20, C21, C23, C24, C25, C26, C27, C28, C3, C4, C5, C6, C7, C76, C77, C78, C79, C8, C80, C81, C86, C9: symbol Device:C -> glasgow-rescue:C-Device
- C87: symbol Device:CP -> glasgow-rescue:CP-Device
- D1, D2, D3, D4, D5: symbol Device:LED -> glasgow-rescue:LED-Device
- FB1: symbol Device:Ferrite_Bead -> glasgow-rescue:Ferrite_Bead-Device
- J1: symbol Connector:USB_C_Receptacle_USB2.0 -> glasgow-rescue:USB_C_Receptacle_USB2.0-Connector
- MK1, MK2, MK3, MK4: symbol Mechanical:MountingHole_Pad -> glasgow-rescue:MountingHole_Pad-Mechanical
- R1, R12, R13, R14, R15, R16, R17, R18, R19, R2, R3, R31, R32, R4, R40, R5, R6, R7, R8, R9: symbol Device:R -> glasgow-rescue:R-Device
- R52, R53: value 5k11 -> 5K1; symbol Device:R -> glasgow-rescue:R-Device
- TP1, TP10, TP11, TP12, TP13, TP14, TP15, TP16, TP17, TP2, TP3, TP4, TP5, TP6, TP7, TP8, TP9: symbol Connector:TestPoint -> glasgow-rescue:TestPoint-Connector
- U1: symbol MCU_Cypress:CY7C68013A-56LTX -> glasgow-rescue:CY7C68013A-56LTX-MCU_Cypress
- U15: symbol Power_Protection:TPD3S014 -> glasgow-rescue:TPD3S014-Power_Protection
- U2: symbol Memory_EEPROM:CAT24M01W -> glasgow-rescue:CAT24M01W-Memory_EEPROM
- U3: symbol Memory_EEPROM:CAT24C256 -> glasgow-rescue:CAT24C256-Memory_EEPROM
- U30: symbol FPGA_Lattice:ICE40HX8K-BG121 -> glasgow-rescue:ICE40HX8K-BG121-FPGA_Lattice
- U7: symbol Power_Supervisor:LM3880 -> glasgow-rescue:LM3880-Power_Supervisor
- Y1: symbol Device:Crystal_GND24 -> glasgow-rescue:Crystal_GND24-Device
