File: hardware/boards/glasgow/io_banks.sch (KiCad schematic (older format))
At the start: 26 parts, among them J10 Conn_01x03, J4 Conn_01x02, J5 Conn_02x22_Odd_Even, U30 ICE40HX8K-BG121, U32 SN74LVC1T45DRL

Commit message: changed level shifters, passing DRC
Parts:
- C33, C85: symbol Device:C -> glasgow-rescue:C-Device
- D10, D6, D7, D8, D9: symbol Device:LED -> glasgow-rescue:LED-Device
- D11, D12, D13: symbol Device:D_Zener -> glasgow-rescue:D_Zener-Device
- J10: symbol Connector_Generic:Conn_01x03 -> glasgow-rescue:Conn_01x03-Connector_Generic
- J4: symbol Connector_Generic:Conn_01x02 -> glasgow-rescue:Conn_01x02-Connector_Generic
- J5: symbol Connector_Generic:Conn_02x22_Odd_Even -> glasgow-rescue:Conn_02x22_Odd_Even-Connector_Generic
- R10, R11, R20, R21, R22, R23, R38, R39, R43, R44, R45: symbol Device:R -> glasgow-rescue:R-Device
- U30: symbol FPGA_Lattice:ICE40HX8K-BG121 -> glasgow-rescue:ICE40HX8K-BG121-FPGA_Lattice
- U32: footprint Glasgow:SOT-563 -> Package_TO_SOT_SMD:SOT-363_SC-70-6; symbol Logic_LevelTranslator:SN74LVC1T45DRL -> glasgow-rescue:SN74LVC1T45DRL-Logic_LevelTranslator
Changed lines of the file:
@@
 QB7
 $Comp
-L power:+3.3V #PWR?
+L glasgow-rescue:+3.3V-power #PWR?
 U 1 1 5C9E33BC
 P 1300 2800
@@
 	6000 4500 6100 4500
 $Comp
-L power:GND #PWR?
+L glasgow-rescue:GND-power #PWR?
 U 1 1 5C9E33C8
 P 6000 4500
@@
 	6000 4600 6100 4600
 $Comp
-L power:GND #PWR?
+L glasgow-rescue:GND-power #PWR?
 U 1 1 5C9E33D4
 P 6000 4600
@@
 	1300 2850 1300 2800
 $Comp
-L FPGA_Lattice:ICE40HX8K-BG121 U?
+L glasgow-rescue:ICE40HX8K-BG121-FPGA_Lattice U?
 U 2 1 5C9E33E2
 P 4750 4450
@@
 $EndComp
 $Comp
-L FPGA_Lattice:ICE40HX8K-BG121 U?
+L glasgow-rescue:ICE40HX8K-BG121-FPGA_Lattice U?
 U 4 1 5C9E33E9
 P 8250 4200
@@
 $EndComp
 $Comp
-L power:+3.3V #PWR?
+L glasgow-rescue:+3.3V-power #PWR?
 U 1 1 5C9E33F0
 P 4750 3050
@@
 VIO_AUX
 $Comp
-L Connector_Generic:Conn_02x22_Odd_Even J?
+L glasgow-rescue:Conn_02x22_Odd_Even-Connector_Generic J?
 U 1 1 5C9E342D
 P 10000 4300
@@
 	9700 3300 9700 3600
 $Comp
-L power:+3.3V #PWR?
+L glasgow-rescue:+3.3V-power #PWR?
 U 1 1 5C9E3436
 P 10550 3200
@@
 	10400 5550 10050 5550
 $Comp
-L power:GND #PWR?
+L glasgow-rescue:GND-power #PWR?
 U 1 1 5C9E343F
 P 10050 5550
@@
 Connection ~ 10400 3500
 $Comp
-L Device:LED D?
+L glasgow-rescue:LED-Device D?
 U 1 1 5C9E3491
 P 9800 1050
@@
 Manually calibrated
 $Comp
-L Device:LED D?
+L glasgow-rescue:LED-Device D?
 U 1 1 5C9E349B
 P 9800 1250
@@
 $EndComp
 $Comp
-L Device:LED D?
+L glasgow-rescue:LED-Device D?
 U 1 1 5C9E34A4
 P 9800 1450
@@
 $EndComp
 $Comp
-L Device:LED D?
+L glasgow-rescue:LED-Device D?
 U 1 1 5C9E34AD
 P 9800 1650
@@
 $EndComp
 $Comp
-L Device:LED D?
+L glasgow-rescue:LED-Device D?
 U 1 1 5C9E34B6
 P 9800 1850
@@
 	10000 1850 10000 1900
 $Comp
-L power:GND #PWR?
+L glasgow-rescue:GND-power #PWR?
 U 1 1 5C9E34C4
 P 10000 1900
@@
 $EndComp
 $Comp
-L Device:R R?
+L glasgow-rescue:R-Device R?
 U 1 1 5C9E34D0
 P 9450 1050
@@
 	9600 1050 9650 1050
 $Comp
-L Device:R R?
+L glasgow-rescue:R-Device R?
 U 1 1 5C9E34DB
 P 9450 1650
@@
 	9650 1850 9600 1850
 $Comp
-L Device:R R?
+L glasgow-rescue:R-Device R?
 U 1 1 5C9E34EB
 P 9450 1850
@@
 $EndComp
 $Comp
-L Device:R R?
+L glasgow-rescue:R-Device R?
 U 1 1 5C9E34F4
 P 9450 1250
@@
 $EndComp
 $Comp
-L Device:R R?
+L glasgow-rescue:R-Device R?
 U 1 1 5C9E34FD
 P 9450 1450
@@
 	5700 4700 6100 4700
 $Comp
-L power:GND #PWR?
+L glasgow-rescue:GND-power #PWR?
 U 1 1 5CDEFF88
 P 2550 4700
@@
 DB7
 $Comp
-L Device:C C?
+L glasgow-rescue:C-Device C?
 U 1 1 5CF06543
 P 8850 2650
@@
 	8850 2500 8850 2450
 $Comp
-L power:GND #PWR?
+L glasgow-rescue:GND-power #PWR?
 U 1 1 5CF0654D
 P 8850 2800
@@
 DA7
 $Comp
-L Connector_Generic:Conn_01x03 J10
+L glasgow-rescue:Conn_01x03-Connector_Generic J10
 U 1 1 5C072C23
 P 3450 3550
@@
 $EndComp
 $Comp
-L power:GND #PWR?
+L glasgow-rescue:GND-power #PWR?
 U 1 1 5C0F528A
 P 3150 3200
@@
 $EndComp
 $Comp
-L Connector_Generic:Conn_01x02 J?
+L glasgow-rescue:Conn_01x02-Connector_Generic J?
 U 1 1 5C961091
 P 4500 2500
@@
 $EndComp
 $Comp
-L power:GND #PWR?
+L glasgow-rescue:GND-power #PWR?
 U 1 1 5C961098
 P 4300 2700
@@
 ~SYNC
 $Comp
-L Device:R R?
+L glasgow-rescue:R-Device R?
 U 1 1 5C9610A4
 P 1950 2750
@@
 $EndComp
 $Comp
-L FPGA_Lattice:ICE40HX8K-BG121 U?
+L glasgow-rescue:ICE40HX8K-BG121-FPGA_Lattice U?
 U 1 1 5C9E33DB
 P 1300 4250
@@
 	9150 1050 9300 1050
 $Comp
-L Logic_LevelTranslator:SN74LVC1T45DRL U32
+L glasgow-rescue:SN74LVC1T45DRL-Logic_LevelTranslator U32
 U 1 1 5CA4F297
 P 2650 2400
 F 0 "U32" H 2850 2850 50  0000 L CNN
 F 1 "SN74LVC1T45DRL" H 2850 2750 50  0000 L CNN
-F 2 "Glasgow:SOT-563" H 2650 1950 50  0001 C CNN
+F 2 "Package_TO_SOT_SMD:SOT-363_SC-70-6" H 2650 1950 50  0001 C CNN
 F 3 "http://www.ti.com/lit/ds/symlink/sn74lvc1t45.pdf" H 1750 1750 50  0001 C CNN
 F 4 "Texas Instruments" H 2650 2400 50  0001 C CNN "Mfg"
@@
 	2250 2600 2200 2600
 $Comp
-L power:GND #PWR?
+L glasgow-rescue:GND-power #PWR?
 U 1 1 5CBEC27E
 P 2650 2800
@@
 $EndComp
 $Comp
-L power:+3.3V #PWR?
+L glasgow-rescue:+3.3V-power #PWR?
 U 1 1 5CBEC3EE
 P 2550 1700
@@
 $EndComp
 $Comp
-L power:GND #PWR?
+L glasgow-rescue:GND-power #PWR?
 U 1 1 5CC04643
 P 1950 2950
@@
 	2200 2600 2200 5250
 $Comp
-L Device:C C?
+L glasgow-rescue:C-Device C?
 U 1 1 5CCC4D9E
 P 2100 1900
@@
 $EndComp
 $Comp
-L power:GND #PWR?
+L glasgow-rescue:GND-power #PWR?
 U 1 1 5CCC4E88
 P 2100 2050
@@
 	1850 5150 1850 5800
 $Comp
-L Device:R R?
+L glasgow-rescue:R-Device R?
 U 1 1 5CBF4EC8
 P 3250 2400
@@
 	2550 3550 2700 3550
 $Comp
-L power:PWR_FLAG #FLG0101
+L glasgow-rescue:PWR_FLAG-power #FLG0101
 U 1 1 5CFF6FB6
 P 8550 2450
@@
 	8550 2450 8850 2450
 $Comp
-L Device:D_Zener D11
+L glasgow-rescue:D_Zener-Device D11
 U 1 1 5D1DFDD1
 P 3650 2550
@@
 	3650 2700 4300 2700
 $Comp
-L Device:R R?
+L glasgow-rescue:R-Device R?
 U 1 1 5CB2B53C
 P 3650 2150
@@
 	3650 2300 3650 2400
 $Comp
-L power:+3.3V #PWR?
+L glasgow-rescue:+3.3V-power #PWR?
 U 1 1 5CB44D27
 P 3650 2000
@@
 	2050 5800 3450 5800
 $Comp
-L Device:D_Zener D12
+L glasgow-rescue:D_Zener-Device D12
 U 1 1 5CB8809B
 P 2700 3350
@@
 $EndComp
 $Comp
-L Device:D_Zener D13
+L glasgow-rescue:D_Zener-Device D13
 U 1 1 5CB88F58
 P 3000 3350
@@
 Auxiliary connector that \nmay be used for exper-\nimenting with addons. \nThere is no guarantee \nthat this connector will\nbe kept in future revisions.
 $Comp
-L Device:R R?
+L glasgow-rescue:R-Device R?
 U 1 1 5CB5DA66
 P 2050 2400
@@
 	2200 2400 2250 2400
 $Comp
-L Device:R R?
+L glasgow-rescue:R-Device R?
 U 1 1 5CBF65F8
 P 2400 3650
@@
 $EndComp
 $Comp
-L Device:R R?
+L glasgow-rescue:R-Device R?
 U 1 1 5CBF658E
 P 2400 3550
