File: hardware/boards/glasgow/io_buffer.sch (KiCad schematic (older format))
At the start: 56 parts, among them J2 Conn_02x10_Odd_Even, J6 Conn_01x08, J7 Conn_01x08, U10 DAC081C081CIMK, U11 TPS73101DBV, U16 SN74LVC1T45DRL, U17 SN74LVC1T45DRL, U18 SN74LVC1T45DRL, U19 PCA6408APW, U19 SN74LVC1T45DRL, U20 SN74LVC1T45DRL, U21 SN74LVC1T45DRL, U33 MG2040, U5 SN74LVC1T45DRL, U6 SN74LVC1T45DRL, U9 ADC081C021CIMM

Commit message: changed level shifters, passing DRC
Parts:
- C30, C32, C35, C36, C37, C38, C39, C40, C47, C48, C49, C50, C51, C52, C53, C54, C55, C56, C57, C58, C59, C82, C83, C84: symbol Device:C -> glasgow-rescue:C-Device
- D14: symbol Device:LED -> glasgow-rescue:LED-Device
- J2: symbol Connector_Generic:Conn_02x10_Odd_Even -> glasgow-rescue:Conn_02x10_Odd_Even-Connector_Generic
- J6, J7: symbol Connector_Generic:Conn_01x08 -> glasgow-rescue:Conn_01x08-Connector_Generic
- R20, R21, R22, R23, R24, R37, R42, R46, R49, R51: symbol Device:R -> glasgow-rescue:R-Device
- RN1, RN2, RN6: symbol Device:R_Pack08 -> glasgow-rescue:R_Pack08-Device
- TP19: symbol Connector:TestPoint -> glasgow-rescue:TestPoint-Connector
- U10: symbol Analog_DAC:DAC081C081CIMK -> glasgow-rescue:DAC081C081CIMK-Analog_DAC
- U11: symbol Regulator_Linear:TPS73101DBV -> glasgow-rescue:TPS73101DBV-Regulator_Linear
- U16, U17, U18, U19, U20, U21, U5, U6: footprint Glasgow:SOT-563 -> Package_TO_SOT_SMD:SOT-363_SC-70-6; symbol Logic_LevelTranslator:SN74LVC1T45DRL -> glasgow-rescue:SN74LVC1T45DRL-Logic_LevelTranslator
- U9: symbol Analog_ADC:ADC081C021CIMM -> glasgow-rescue:ADC081C021CIMM-Analog_ADC
